Commit message: update GUI

File: src/robot_description/urdf/materials.xacro (robot description, xacro)
@@ -19,3 +19,59 @@
     <color  rgba  ="0.5 0.5 0.5 1.0"/>
   </material>
+  <!-- material for the robot's body -->
+  <material name  ="base_link">
+    <color rgba="0.216 0.227 0.243 1.0"/>
+  </material>
+  <material name  ="link_1">
+    <color  rgba  ="0.569 0.588 0.608 1.0"/>
+  </material>
+  <material name  ="link_2">
+    <color  rgba  ="0.471 0.49 0.51 1.0"/>
+  </material>
+  <material name  ="link_3">
+    <color  rgba  ="0.569 0.588 0.608 1.0"/>
+  </material>
+  <material name  ="link_4">
+    <color  rgba  ="0.471 0.49 0.51 1.0"/>
+  </material>
+  <material name  ="link_5">
+    <color  rgba  ="0.569 0.588 0.608 1.0"/>
+  </material>
+  <material name  ="tool_flange">
+    <color rgba="0.569 0.588 0.608 1.0"/>
+  </material>
+  <material name  ="tool">
+    <color  rgba  ="0.439 0.417 0.502 1.0"/>
+  </material>
+  <!-- material for the robot's body -->
+  <material name  ="body">
+    <color rgba="0.471 0.490 0.510 1.0"/>
+  </material>
+  <material name  ="link">
+    <color rgba="0.275 0.290 0.306 1.0"/>
+  </material>
+  <material name  ="robot_base">
+   <color rgba="0.216 0.227 0.243 1.0"/>
+  </material>
+  <material name  ="robot_abb">
+    <color  rgba  ="0.5 0.5 0.5 1.0"/>
+  </material>
+  <material name  ="robot_fanuc">
+    <color  rgba  ="0.5 0.5 0.5 1.0"/>
+  </material>
+  <material name  ="robot_kuka">
+    <color  rgba  ="0.5 0.5 0.5 1.0"/>
+  </material>
+  <material name  ="light_gunmetal">
+    <color  rgba  ="0.471 0.49 0.51 1.0"/>
+  </material>
+  <material name  ="titanium">
+    <color  rgba  ="0.569 0.588 0.608 1.0"/>
+  </material>
+  <material name  ="dark_silver">
+    <color  rgba  ="0.529 0.541 0.557 1.0"/>
+  </material>
+  <material name  ="slate_ray">
+    <color  rgba  ="0.439 0.417 0.502 1.0"/>
+  </material>
 </robot>

File: src/robot_description/urdf/robot.xacro (robot description, xacro)
@@ -23,5 +23,5 @@
         <mesh filename  ="package://robot_description/meshes/base_link.stl" />
       </geometry>
-      <material   name  ="grey"></material>
+      <material   name  ="base_link"></material>
     </visual>
     <collision>
@@ -50,5 +50,5 @@
         <mesh filename  ="package://robot_description/meshes/link_1.stl" />
       </geometry>
-      <material   name  ="grey"></material>
+      <material   name  ="link_1"></material>
     </visual>
     <collision>
@@ -77,5 +77,5 @@
         <mesh   filename ="package://robot_description/meshes/link_2.stl" />
       </geometry>
-      <material     name  ="grey"></material>
+      <material     name  ="link_2"></material>
     </visual>
     <collision>
@@ -104,5 +104,5 @@
         <mesh  filename="package://robot_description/meshes/link_3.stl" />
       </geometry>
-      <material name="grey"></material>
+      <material name="link_3"></material>
     </visual>
     <collision>
@@ -131,5 +131,5 @@
         <mesh filename="package://robot_description/meshes/link_4.stl" />
       </geometry>
-      <material name="grey"></material>
+      <material name="link_4"></material>
     </visual>
     <collision>
@@ -158,5 +158,5 @@
         <mesh filename  ="package://robot_description/meshes/link_5.stl" />
       </geometry>
-      <material   name  ="grey"></material>
+      <material   name  ="link_5"></material>
     </visual>
     <collision>
@@ -185,5 +185,5 @@
         <mesh filename  ="package://robot_description/meshes/link_6.stl" />
       </geometry>
-      <material   name  ="grey"></material>
+      <material   name  ="tool_flange"></material>
     </visual>
     <collision>
@@ -213,5 +213,5 @@
         <mesh filename  ="package://robot_description/meshes/gripper_l.stl" />
       </geometry>
-      <material   name  ="grey"></material>
+      <material   name  ="tool"></material>
     </visual>
     <collision>
@@ -240,5 +240,5 @@
         <mesh filename  ="package://robot_description/meshes/gripper_r.stl" />
       </geometry>
-      <material   name  ="grey"></material>
+      <material   name  ="tool"></material>
     </visual>
     <collision>
