Commit message: pkg pick_place

File: src/robot_description/urdf/robot.urdf.xacro (robot description, xacro)
@@ -12,7 +12,7 @@
     <xacro:base_camera
             parent_link     ="base_link"
-            base_link       ="astra_link"
+            base_link       ="astra_base"
             camera_name     ="astra_depth"
-            frame_name      ="astra_link"/>
+            frame_name      ="astra"/>
     <xacro:robot_ros2_control
             name                    ="robot"

File: src/robot_description/urdf/robot.xacro (robot description, xacro)
@@ -26,7 +26,7 @@
     </visual>
     <collision>
-      <origin xyz ="0 0 0" rpy ="0 0 0" />
-      <geometry>
-        <mesh filename  ="package://robot_description/meshes/base_link.stl" />
+      <origin xyz ="-0.05 0 0.03" rpy ="0 0 0" />
+      <geometry>
+        <box size="0.2 0.15 0.06"/>
       </geometry>
     </collision>
@@ -53,7 +53,7 @@
     </visual>
     <collision>
-      <origin xyz ="0 0 0" rpy  ="0 0 0" />
-      <geometry>
-        <mesh filename  ="package://robot_description/meshes/link_1.stl" />
+      <origin xyz ="0 0 0.15" rpy  ="0 0 0" />
+      <geometry>
+        <cylinder radius="0.17" length="0.3"/>
       </geometry>
     </collision>
@@ -80,7 +80,7 @@
     </visual>
     <collision>
-      <origin xyz="0 0 0" rpy="0 0 0" />
-      <geometry>
-        <mesh filename="package://robot_description/meshes/link_2.stl" />
+      <origin xyz="0.15 0 -0.05" rpy="0 0 0" />
+      <geometry>
+         <box size="0.3 0.12 0.1"/>
       </geometry>
     </collision>
@@ -107,7 +107,7 @@
     </visual>
     <collision>
-      <origin  xyz="0 0 0" rpy="0 0 0" />
-      <geometry>
-        <mesh  filename="package://robot_description/meshes/link_3.stl" />
+      <origin  xyz="0 -0.08 -0.05" rpy="0 0 0" />
+      <geometry>
+        <box size="0.16 0.16 0.1"/>
       </geometry>
     </collision>
@@ -134,7 +134,7 @@
     </visual>
     <collision>
-      <origin  xyz="0 0 0"  rpy="0 0 0" />
-      <geometry>
-        <mesh filename="package://robot_description/meshes/link_4.stl" />
+      <origin  xyz="0 0 0.1" rpy="0 0 0" />
+      <geometry>
+        <box size="0.1 0.1 0.2"/>
       </geometry>
     </collision>
@@ -161,7 +161,7 @@
     </visual>
     <collision>
-      <origin  xyz="0 0 0"  rpy="0 0 0" />
-      <geometry>
-        <mesh filename  ="package://robot_description/meshes/link_5.stl" />
+      <origin  xyz="0 0 -0.04" rpy="0 0 0" />
+      <geometry>
+        <box size="0.2 0.08 0.08"/>
       </geometry>
     </collision>
@@ -188,7 +188,7 @@
     </visual>
     <collision>
-      <origin  xyz  ="0 0 0"  rpy ="0 0 0" />
-      <geometry>
-        <mesh filename  ="package://robot_description/meshes/link_6.stl" />
+      <origin  xyz="0 0 0.05" rpy="0 0 0" />
+      <geometry>
+        <box size="0.11 0.04 0.06"/>
       </geometry>
     </collision>
@@ -216,7 +216,7 @@
     </visual>
     <collision>
-      <origin xyz="0 0 0" rpy="0 0 0" />
-      <geometry>
-        <mesh filename  ="package://robot_description/meshes/gripper_l.stl" />
+      <origin xyz="0.006 0 0.015" rpy="0 0 0" />
+      <geometry>
+        <box size="0.01 0.02 0.03"/>
       </geometry>
     </collision>
@@ -243,7 +243,7 @@
     </visual>
     <collision>
-      <origin xyz ="0 0 0" rpy  ="0 0 0" />
-      <geometry>
-        <mesh  filename ="package://robot_description/meshes/gripper_r.stl" />
+      <origin xyz="0.006 0 0.015" rpy="0 0 0" />
+      <geometry>
+        <box size="0.01 0.02 0.03"/>
       </geometry>
     </collision>

File: src/robot_description/urdf/sensors.xacro (robot description, xacro)
@@ -24,22 +24,23 @@
       </collision>
     </link>
-    <link           name  ="${base_link}_optical"/>
+    <link           name  ="${frame_name}_optical"/>
     <joint          name  ="${base_link}_joint"         type  ="fixed">
       <parent       link  ="${parent_link}"/>
       <child        link  ="${base_link}"/>
-      <origin       xyz   ="0.6 0 1.0" rpy="${pi} 0 ${pi/2}"/>
+      <origin       xyz   ="0.7 0 0.9" rpy="${pi} ${pi/12} 0"/>
     </joint>
+    <!-- rpy= ${pi} ${pi/12} 0-->
     <joint          name  ="${base_link}_optical_joint" type  ="fixed">
       <parent       link  ="${base_link}"/>
-      <child        link  ="${base_link}_optical"/>
+      <child        link  ="${frame_name}_optical"/>
       <origin       xyz   ="0 0 0" rpy="0 0 0"/>
     </joint>
-    <gazebo reference="${base_link}">
+    <gazebo reference="${frame_name}_optical">
       <sensor name="astra_rgb" type="camera">
-        <pose>0 0 0 0 ${-pi/2} ${pi} </pose>
+        <pose>0 0 0  0  ${-pi/2} ${pi/2}  </pose>
         <always_on>true</always_on>
         <update_rate>20</update_rate>
         <visualize>true</visualize>
-        <topic>astra/rgb/image_raw</topic>
+        <topic>astra_sim/rgb/image_raw</topic>
         <camera>
           <image>
@@ -55,11 +56,11 @@
       </sensor>
     </gazebo>
-    <gazebo reference="${base_link}">
+    <gazebo reference="${frame_name}_optical">
       <sensor name="astra_depth" type="depth">
-        <pose>0 0 0 0 ${-pi/2} 0</pose>
+        <pose>0 0 0  0  ${-pi/2} ${pi/2}  </pose>
         <always_on>true</always_on>
         <update_rate>20</update_rate>
         <visualize>true</visualize>
-        <topic>astra/depth/image_raw</topic>
+        <topic>astra_sim/depth/image_raw</topic>
         <camera>
           <image>

Commit message: Clearn Action

File: src/robot_description/urdf/robot.urdf.xacro (robot description, xacro)
@@ -6,5 +6,5 @@
             default ="$(find robot_control)/config/initial_positions.yaml" />
     <xacro:include filename ="$(find robot_description)/urdf/materials.xacro" />
-    <xacro:include filename ="$(find robot_description)/urdf/robot.xacro" />
+    <xacro:include filename ="$(find robot_description)/urdf/robot_tcp_xy.xacro" /> <!-- robot.xacro  |robot_tcp_z.xacro | robot_tcp_xy.xacro-->
     <xacro:include filename ="$(find robot_description)/urdf/sensors.xacro"/>
     <xacro:include filename ="$(find robot_description)/urdf/ros2_control.xacro" />

File: src/robot_description/urdf/robot_tcp_xy.xacro (robot description, xacro)
@@ -181,7 +181,7 @@
     </inertial>
     <visual>
-      <origin xyz ="0 0 0" rpy  ="0 0 0" />
-      <geometry>
-        <mesh filename  ="package://robot_description/meshes/link_6.stl" />
+      <origin xyz ="0 0 0" rpy  ="0 0 ${pi}" />
+      <geometry>
+        <mesh filename  ="package://robot_description/meshes/tcp_xy.stl" />
       </geometry>
       <material   name  ="tool_flange"></material>
@@ -190,5 +190,5 @@
       <origin xyz ="0 0 0" rpy ="0 0 0" />
       <geometry>
-        <mesh filename  ="package://robot_description/meshes/dae/link_6.dae" />
+        <mesh filename  ="package://robot_description/meshes/tcp_xy.stl" />
       </geometry>
     </collision>
@@ -213,5 +213,5 @@
         <mesh filename  ="package://robot_description/meshes/gripper_l.stl" />
       </geometry>
-      <material   name  ="tool"></material>
+      <material   name  ="gripper_l"></material>
     </visual>
     <collision>
@@ -240,5 +240,5 @@
         <mesh filename  ="package://robot_description/meshes/gripper_r.stl" />
       </geometry>
-      <material   name  ="tool"></material>
+      <material   name  ="gripper_r"></material>
     </visual>
     <collision>
@@ -257,5 +257,5 @@
   </joint>
   <joint    name  ="tcp_joint"             type      ="fixed">
-    <origin xyz   ="0 0 0.08"              rpy       ="0 0 0"/>
+    <origin xyz   ="0 0.036 0.021"              rpy       ="0 0 0"/>
     <parent link  ="link_6"/>
     <child  link  ="tcp_link"/>
@@ -317,5 +317,5 @@
   <!-- joint_gl -->
   <joint    name  ="joint_gl"              type      ="prismatic">
-    <origin xyz   ="0.0021 0 0.0668"       rpy       ="0 0 0" />
+    <origin xyz   ="0.0021 0 -0.0668"       rpy       ="0 0 0" />
     <parent link  ="link_6" />
     <child  link  ="gripper_l" />
@@ -326,5 +326,5 @@
   <!-- joint_gr -->
   <joint    name  ="joint_gr"              type      ="prismatic">
-    <origin xyz   ="-0.0021 0 0.0668"      rpy       ="0 0 ${pi}" />
+    <origin xyz   ="-0.0021 0 -0.0668"      rpy       ="0 0 ${pi}" />
     <parent link  ="link_6" />
     <child  link  ="gripper_r" />

File: src/robot_description/urdf/robot_tcp_z.xacro (robot description, xacro)
@@ -23,5 +23,5 @@
         <mesh filename  ="package://robot_description/meshes/base_link.stl" />
       </geometry>
-      <material   name  ="black"></material>
+      <material   name  ="base_link"></material>
     </visual>
     <collision>
@@ -50,5 +50,5 @@
         <mesh filename  ="package://robot_description/meshes/link_1.stl" />
       </geometry>
-      <material   name  ="blue"></material>
+      <material   name  ="link_1"></material>
     </visual>
     <collision>
@@ -77,5 +77,5 @@
         <mesh   filename ="package://robot_description/meshes/link_2.stl" />
       </geometry>
-      <material     name  ="grey"></material>
+      <material     name  ="link_2"></material>
     </visual>
     <collision>
@@ -104,5 +104,5 @@
         <mesh  filename="package://robot_description/meshes/link_3.stl" />
       </geometry>
-      <material name="blue"></material>
+      <material name="link_3"></material>
     </visual>
     <collision>
@@ -131,5 +131,5 @@
         <mesh filename="package://robot_description/meshes/link_4.stl" />
       </geometry>
-      <material name="grey"></material>
+      <material name="link_4"></material>
     </visual>
     <collision>
@@ -158,5 +158,5 @@
         <mesh filename  ="package://robot_description/meshes/link_5.stl" />
       </geometry>
-      <material   name  ="blue"></material>
+      <material   name  ="link_5"></material>
     </visual>
     <collision>
@@ -185,5 +185,5 @@
         <mesh filename  ="package://robot_description/meshes/tcp_z.stl" />
       </geometry>
-      <material   name  ="grey"></material>
+      <material   name  ="tool_flange"></material>
     </visual>
     <collision>
@@ -213,5 +213,5 @@
         <mesh filename  ="package://robot_description/meshes/gripper_l.stl" />
       </geometry>
-      <material   name  ="grey"></material>
+      <material   name  ="gripper_l"></material>
     </visual>
     <collision>
@@ -240,5 +240,5 @@
         <mesh filename  ="package://robot_description/meshes/gripper_r.stl" />
       </geometry>
-      <material   name  ="grey"></material>
+      <material   name  ="gripper_r"></material>
     </visual>
     <collision>
@@ -308,9 +308,9 @@
   <!-- JOINT 6 -->
   <joint    name  ="joint_6"               type    ="revolute">
-    <origin xyz   ="0.132 0 -0.05"      rpy     ="0 ${-pi/2} ${pi}" />
+    <origin xyz   ="0.132 0 -0.05"      rpy        = "0 ${pi/2} 0  " />
     <parent link  ="link_5" />
     <child  link  ="link_6" />
     <axis   xyz   ="0 0 1" />
-    <limit  lower ="-1.5707"               upper     ="1.5707"
+    <limit  lower ="-3.14159"               upper     ="3.14159"
             effort="1000"                  velocity  ="5.0" />
   </joint>
