Commit message: demo Drl Path

File: src/robot_description/urdf/robot.xacro (robot description, xacro)
@@ -26,7 +26,7 @@
     </visual>
     <collision>
-      <origin xyz ="-0.05 0 0.03" rpy ="0 0 0" />
-      <geometry>
-        <box size="0.2 0.15 0.06"/>
+      <origin xyz ="0 0 0" rpy ="0 0 0" />
+      <geometry>
+        <mesh filename  ="package://robot_description/meshes/dae/base_link.dae" />
       </geometry>
     </collision>
@@ -53,7 +53,7 @@
     </visual>
     <collision>
-      <origin xyz ="0 0 0.15" rpy  ="0 0 0" />
-      <geometry>
-        <cylinder radius="0.17" length="0.3"/>
+      <origin xyz ="0 0 0" rpy ="0 0 0" />
+      <geometry>
+        <mesh filename  ="package://robot_description/meshes/dae/link_1.dae" />
       </geometry>
     </collision>
@@ -80,7 +80,7 @@
     </visual>
     <collision>
-      <origin xyz="0.15 0 -0.05" rpy="0 0 0" />
-      <geometry>
-         <box size="0.3 0.12 0.1"/>
+      <origin xyz ="0 0 0" rpy ="0 0 0" />
+      <geometry>
+        <mesh filename  ="package://robot_description/meshes/dae/link_2.dae" />
       </geometry>
     </collision>
@@ -107,7 +107,7 @@
     </visual>
     <collision>
-      <origin  xyz="0 -0.08 -0.05" rpy="0 0 0" />
-      <geometry>
-        <box size="0.16 0.16 0.1"/>
+      <origin xyz ="0 0 0" rpy ="0 0 0" />
+      <geometry>
+        <mesh filename  ="package://robot_description/meshes/dae/link_3.dae" />
       </geometry>
     </collision>
@@ -134,7 +134,7 @@
     </visual>
     <collision>
-      <origin  xyz="0 0 0.1" rpy="0 0 0" />
-      <geometry>
-        <box size="0.1 0.1 0.2"/>
+      <origin xyz ="0 0 0" rpy ="0 0 0" />
+      <geometry>
+        <mesh filename  ="package://robot_description/meshes/dae/link_4.dae" />
       </geometry>
     </collision>
@@ -161,7 +161,7 @@
     </visual>
     <collision>
-      <origin  xyz="0 0 -0.04" rpy="0 0 0" />
-      <geometry>
-        <box size="0.2 0.08 0.08"/>
+      <origin xyz ="0 0 0" rpy ="0 0 0" />
+      <geometry>
+        <mesh filename  ="package://robot_description/meshes/dae/link_5.dae" />
       </geometry>
     </collision>
@@ -188,7 +188,7 @@
     </visual>
     <collision>
-      <origin  xyz="0 0 0.05" rpy="0 0 0" />
-      <geometry>
-        <box size="0.11 0.04 0.06"/>
+      <origin xyz ="0 0 0" rpy ="0 0 0" />
+      <geometry>
+        <mesh filename  ="package://robot_description/meshes/dae/link_6.dae" />
       </geometry>
     </collision>
@@ -216,7 +216,7 @@
     </visual>
     <collision>
-      <origin xyz="0.006 0 0.015" rpy="0 0 0" />
-      <geometry>
-        <box size="0.01 0.02 0.03"/>
+      <origin xyz ="0 0 0" rpy ="0 0 0" />
+      <geometry>
+        <mesh filename  ="package://robot_description/meshes/dae/gripper_l.dae" />
       </geometry>
     </collision>
@@ -243,7 +243,7 @@
     </visual>
     <collision>
-      <origin xyz="0.006 0 0.015" rpy="0 0 0" />
-      <geometry>
-        <box size="0.01 0.02 0.03"/>
+      <origin xyz ="0 0 0" rpy ="0 0 0" />
+      <geometry>
+        <mesh filename  ="package://robot_description/meshes/dae/gripper_r.dae" />
       </geometry>
     </collision>

Commit message: GUI_Rviz

File: src/robot_description/urdf/robot.xacro (robot description, xacro)
@@ -23,5 +23,5 @@
         <mesh filename  ="package://robot_description/meshes/base_link.stl" />
       </geometry>
-      <material   name  ="white"></material>
+      <material   name  ="grey"></material>
     </visual>
     <collision>
@@ -50,5 +50,5 @@
         <mesh filename  ="package://robot_description/meshes/link_1.stl" />
       </geometry>
-      <material   name  ="white"></material>
+      <material   name  ="grey"></material>
     </visual>
     <collision>
@@ -77,5 +77,5 @@
         <mesh   filename ="package://robot_description/meshes/link_2.stl" />
       </geometry>
-      <material     name  ="white"></material>
+      <material     name  ="grey"></material>
     </visual>
     <collision>
@@ -104,5 +104,5 @@
         <mesh  filename="package://robot_description/meshes/link_3.stl" />
       </geometry>
-      <material name="white"></material>
+      <material name="grey"></material>
     </visual>
     <collision>
@@ -131,5 +131,5 @@
         <mesh filename="package://robot_description/meshes/link_4.stl" />
       </geometry>
-      <material name="white"></material>
+      <material name="grey"></material>
     </visual>
     <collision>
@@ -158,5 +158,5 @@
         <mesh filename  ="package://robot_description/meshes/link_5.stl" />
       </geometry>
-      <material   name  ="white"></material>
+      <material   name  ="grey"></material>
     </visual>
     <collision>
@@ -185,5 +185,5 @@
         <mesh filename  ="package://robot_description/meshes/link_6.stl" />
       </geometry>
-      <material   name  ="white"></material>
+      <material   name  ="grey"></material>
     </visual>
     <collision>
@@ -213,5 +213,5 @@
         <mesh filename  ="package://robot_description/meshes/gripper_l.stl" />
       </geometry>
-      <material   name  ="white"></material>
+      <material   name  ="grey"></material>
     </visual>
     <collision>
@@ -240,5 +240,5 @@
         <mesh filename  ="package://robot_description/meshes/gripper_r.stl" />
       </geometry>
-      <material   name  ="white"></material>
+      <material   name  ="grey"></material>
     </visual>
     <collision>

Commit message: tasks server

File: src/robot_description/urdf/robot.xacro (robot description, xacro)
@@ -321,6 +321,6 @@
     <child  link  ="gripper_l" />
     <axis   xyz   ="1 0 0" />
-    <limit  lower ="-0.001"                upper     ="0.02"
-            effort="50"                    velocity  ="0.05" />
+    <limit  lower ="-0.001"                upper     ="0.025"
+            effort="50"                    velocity  ="0.5" />
   </joint>
   <!-- joint_gr -->
@@ -330,6 +330,6 @@
     <child  link  ="gripper_r" />
     <axis   xyz   ="1 0 0" />
-    <limit  lower ="-0.001"                upper     ="0.02"
-            effort="50"                    velocity  ="0.05" />
+    <limit  lower ="-0.001"                upper     ="0.025"
+            effort="50"                    velocity  ="0.5" />
   </joint>
   <gazebo reference="gripper_l">
